File: pcb/thermostat/_autosave-thermostat.kicad_sch (KiCad schematic)
At the start: 8 parts, among them SW1 RotaryEncoder, SW2 RotaryEncoder_Switch, U1 WeMos_D1_mini, U2 DHT11, U3 ESP32-C3-WROOM-02-H4

Commit message: Added esp32
Parts:
- removed C1: 10nF, Capacitor_SMD:C_0805_2012Metric_Pad1.18x1.45mm_HandSolder, symbol Device:C
- removed SW1: RotaryEncoder, Rotary_Encoder:RotaryEncoder_Alps_EC11E-Switch_Vertical_H20mm, symbol Device:RotaryEncoder
- removed U1: WeMos_D1_mini, Module:WEMOS_D1_mini_light, symbol MCU_Module:WeMos_D1_mini
Connections:
- net +3.3V is gone; now on net +3V3: Brd1.2 (VCC)
- net +5V is gone; now on net +3V3: R1.1, U2.1 (VCC)
- net D+: now also U3.14 (IO19); no longer U3.13 (IO18)
- net D-: now also U3.13 (IO18); no longer U3.14 (IO19)
- net GND: now also U3.19 (GND), U3.20 (GND), U3.21 (GND), U3.22 (GND), U3.23 (GND), U3.24 (GND), U3.25 (GND), U3.26 (GND), U3.27 (GND), U3.28 (GND), U3.29 (GND), U3.30 (GND), U3.31 (GND), U3.32 (GND), U3.33 (GND), U3.34 (GND), U3.35 (GND), U3.36 (GND), U3.37 (GND), U3.38 (GND), U3.39 (GND), U3.9 (GND)
- net +3V3: now reaches U3.1 (3V3)
