File: pcb/thermostat/thermostat.kicad_pcb (KiCad board)
At the start: 2 copper layers, 40.5 x 51.4 mm, 6 parts, among them SW1 RotaryEncoder, U1 WeMos_D1_mini, U2 DHT11

Commit message: Added esp32
Parts:
- removed C1: 10nF, Capacitor_SMD:C_0805_2012Metric_Pad1.18x1.45mm_HandSolder
- removed SW1: RotaryEncoder, Rotary_Encoder:RotaryEncoder_Alps_EC11E-Switch_Vertical_H20mm
- removed U1: WeMos_D1_mini, Module:WEMOS_D1_mini_light
- added U3: ESP32-C3-WROOM-02-H4, esp32-c3:MODULE_ESP32-C3-WROOM-02-H4, F.Cu at (91.3, 109.5)
- moved Brd1 56.4 mm to (66.7, 42.9)
- moved U2 55.5 mm to (116.7, 56.8)
- moved R1 33.4 mm to (134.9, 113.5)
Connections:
- Brd1 pad 2: +3.3V -> +3V3
- R1 pad 1: +5V -> +3V3
- U2 pad 1: +5V -> +3V3
Routing:
- net +5V: track 42.7 -> 0.00 mm
- net +3.3V: track 22.1 -> 0.00 mm
- net RotB: track 15.1 -> 0.00 mm
- net SCL: track 11.5 -> 0.00 mm
- net RotA: track 9.01 -> 0.00 mm
- net SDA: track 8.93 -> 0.00 mm
- net dhtData: track 6.86 -> 0.00 mm
- net GND: track 2.19 -> 0.00 mm, vias 1 -> 0
